File: FC-TxROM-AX5202P.kicad_pcb (KiCad board)
At the start: 2 copper layers, 100.1 x 67.3 mm, 28 parts, among them J1 FAMICOM_EDGE, Q1 2N3904, U1 PRG ROM, U2 CHR ROM/RAM, U3 AX5202P, U4 PRG RAM

Commit message: Release v1.1.0
Parts:
- added R3: 27k, Resistor_THT:R_Axial_DIN0204_L3.6mm_D1.6mm_P7.62mm_Horizontal, F.Cu at (44.5, 66.7)
- JP3, JP4: value Jumper_3_Open -> TKSROM/TLSROM/OTHER
- JP6, JP7: value Jumper_3_Open -> EPROM/FLASH
- JP8: value Jumper_2_Open -> UNSAFE_CE
- JP9: value Jumper_2_Open -> SRAM_VCC
- moved C5 2.54 mm to (42.5, 63.5)
Connections:
- net /PRG_RAM_VCC renamed SRAM_VCC
Routing:
- net GND: track 379.8 -> 383.9 mm
- net /PRG_A16: track 92.9 -> 93.8 mm
