File: FC-TxROM-AX5202P.kicad_sch (KiCad schematic)
At the start: 28 parts, among them J1 FAMICOM_EDGE, Q1 2N3904, U1 PRG ROM, U2 CHR ROM/RAM, U3 AX5202P, U4 PRG RAM, U5 CHR RAM

Commit message: Release v1.1.0
Parts:
- added R3: 27k, Resistor_THT:R_Axial_DIN0204_L3.6mm_D1.6mm_P7.62mm_Horizontal, symbol Device:R
- JP3, JP4: value Jumper_3_Open -> TKSROM/TLSROM/OTHER
- JP6, JP7: value Jumper_3_Open -> EPROM/FLASH
- JP8: value Jumper_2_Open -> UNSAFE_CE
- JP9: value Jumper_2_Open -> SRAM_VCC
Connections:
- net GND: now also R3.1
- net M2: now also R3.2
- net PRG_RAM_VCC renamed SRAM_VCC
Other:
- note added: "32-pin CHR ROM or RAM"
- note added: "CHR ROM or RAM Selection"
- note added: "Decoupling Capacitors"
- note added: "Edge Connector"
- note added: "Mapper"
- note added: "PRG RAM"
- note added: "PRG ROM"
- note added: "Pinout reference only. Not populated / not a physical part. Shows the 28-pin alternative package; U2 is the 32-pin package."
- note added: "SRAM battery backup power circuit"
- note added: "SRAM no-battery power jumpers"
- note added: "TKSROM/TLSROM or Other Board Type Selection"
- note added: "UV EPROM or EEPROM/FLASH Selection"
- moved on the sheet: BT1, C1, C2, C3, C4, C5, C8, D1, D2, JP1, JP3, JP4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
